File: sensorboard/sensorboard.sch (KiCad schematic (older format))
At the start: 12 parts, among them P1 CONN_01X04, U1 LP38691, U2 MCP9808, U3 ABPMANN030PG2A3

Commit message: Finished layout of sensor board
Parts:
- C1, C2, C3, C4: footprint (none) -> Capacitors_SMD:C_0603
- P1: footprint (none) -> footprint:0855025005
- R1, R2, R3, R4: footprint (none) -> Resistors_SMD:R_0603
- U1: footprint (none) -> Housings_DFN_QFN:DFN-6-1EP_3x3mm_Pitch0.95mm
- U2: footprint (none) -> Housings_DFN_QFN:DFN-8-1EP_3x2mm_Pitch0.5mm
- U3: footprint (none) -> footprint:ABPMANN030PG2A3
Changed lines of the file:
@@
 F 0 "U1" H 4850 1550 60  0000 C CNN
 F 1 "LP38691" H 5450 1000 60  0000 C CNN
-F 2 "" H 5150 1300 60  0000 C CNN
+F 2 "Housings_DFN_QFN:DFN-6-1EP_3x3mm_Pitch0.95mm" H 5150 1300 60  0001 C CNN
 F 3 "" H 5150 1300 60  0000 C CNN
 	1    5150 1300
@@
 F 0 "P1" H 1350 3250 50  0000 C CNN
 F 1 "CONN_01X04" V 1450 3000 50  0000 C CNN
-F 2 "" H 1350 3000 50  0000 C CNN
+F 2 "footprint:0855025005" H 1350 3000 50  0001 C CNN
 F 3 "" H 1350 3000 50  0000 C CNN
 	1    1350 3000
@@
 $EndComp
 $Comp
-L +5V #PWR1
+L +5V #PWR01
 U 1 1 5780FAF2
 P 1600 2750
-F 0 "#PWR1" H 1600 2600 50  0001 C CNN
+F 0 "#PWR01" H 1600 2600 50  0001 C CNN
 F 1 "+5V" H 1600 2890 50  0000 C CNN
 F 2 "" H 1600 2750 50  0000 C CNN
@@
 $EndComp
 $Comp
-L GND #PWR2
+L GND #PWR02
 U 1 1 5780FB9B
 P 1600 3250
-F 0 "#PWR2" H 1600 3000 50  0001 C CNN
+F 0 "#PWR02" H 1600 3000 50  0001 C CNN
 F 1 "GND" H 1600 3100 50  0000 C CNN
 F 2 "" H 1600 3250 50  0000 C CNN
@@
 $EndComp
 $Comp
-L +5V #PWR5
+L +5V #PWR03
 U 1 1 5780FC6B
 P 4200 1100
-F 0 "#PWR5" H 4200 950 50  0001 C CNN
+F 0 "#PWR03" H 4200 950 50  0001 C CNN
 F 1 "+5V" H 4200 1240 50  0000 C CNN
 F 2 "" H 4200 1100 50  0000 C CNN
@@
 $EndComp
 $Comp
-L GND #PWR11
+L GND #PWR04
 U 1 1 5780FC7C
 P 5150 1800
-F 0 "#PWR11" H 5150 1550 50  0001 C CNN
+F 0 "#PWR04" H 5150 1550 50  0001 C CNN
 F 1 "GND" H 5150 1650 50  0000 C CNN
 F 2 "" H 5150 1800 50  0000 C CNN
@@
 F 0 "C1" H 4225 1550 50  0000 L CNN
 F 1 "2.2u" H 4225 1350 50  0000 L CNN
-F 2 "" H 4238 1300 50  0000 C CNN
+F 2 "Capacitors_SMD:C_0603" H 4238 1300 50  0001 C CNN
 F 3 "" H 4200 1450 50  0000 C CNN
 	1    4200 1450
@@
 F 0 "C2" H 6225 1550 50  0000 L CNN
 F 1 "2.2u" H 6225 1350 50  0000 L CNN
-F 2 "" H 6238 1300 50  0000 C CNN
+F 2 "Capacitors_SMD:C_0603" H 6238 1300 50  0001 C CNN
 F 3 "" H 6200 1450 50  0000 C CNN
 	1    6200 1450
@@
 Connection ~ 4200 1200
 $Comp
-L GND #PWR6
+L GND #PWR05
 U 1 1 5780FDC8
 P 4200 1650
-F 0 "#PWR6" H 4200 1400 50  0001 C CNN
+F 0 "#PWR05" H 4200 1400 50  0001 C CNN
 F 1 "GND" H 4200 1500 50  0000 C CNN
 F 2 "" H 4200 1650 50  0000 C CNN
@@
 Connection ~ 5750 1200
 $Comp
-L GND #PWR15
+L GND #PWR06
 U 1 1 5780FF17
 P 6200 1650
-F 0 "#PWR15" H 6200 1400 50  0001 C CNN
+F 0 "#PWR06" H 6200 1400 50  0001 C CNN
 F 1 "GND" H 6200 1500 50  0000 C CNN
 F 2 "" H 6200 1650 50  0000 C CNN
@@
 	6200 1650 6200 1600
 $Comp
-L +3.3V #PWR14
+L +3.3V #PWR07
 U 1 1 5780FF8B
 P 6200 1100
-F 0 "#PWR14" H 6200 950 50  0001 C CNN
+F 0 "#PWR07" H 6200 950 50  0001 C CNN
 F 1 "+3.3V" H 6200 1240 50  0000 C CNN
 F 2 "" H 6200 1100 50  0000 C CNN
@@
 	1550 3050 2650 3050
 $Comp
-L +3.3V #PWR12
+L +3.3V #PWR08
 U 1 1 578104BC
 P 5700 2800
-F 0 "#PWR12" H 5700 2650 50  0001 C CNN
+F 0 "#PWR08" H 5700 2650 50  0001 C CNN
 F 1 "+3.3V" H 5700 2940 50  0000 C CNN
 F 2 "" H 5700 2800 50  0000 C CNN
@@
 $EndComp
 $Comp
-L GND #PWR13
+L GND #PWR09
 U 1 1 578104D6
 P 5700 3300
-F 0 "#PWR13" H 5700 3050 50  0001 C CNN
+F 0 "#PWR09" H 5700 3050 50  0001 C CNN
 F 1 "GND" H 5700 3150 50  0000 C CNN
 F 2 "" H 5700 3300 50  0000 C CNN
@@
 $EndComp
 $Comp
-L GND #PWR8
+L GND #PWR010
 U 1 1 578104F0
 P 4600 3400
-F 0 "#PWR8" H 4600 3150 50  0001 C CNN
+F 0 "#PWR010" H 4600 3150 50  0001 C CNN
 F 1 "GND" H 4600 3250 50  0000 C CNN
 F 2 "" H 4600 3400 50  0000 C CNN
@@
 F 0 "C3" H 6525 3150 50  0000 L CNN
 F 1 "0.1u" H 6525 2950 50  0000 L CNN
-F 2 "" H 6538 2900 50  0000 C CNN
+F 2 "Capacitors_SMD:C_0603" H 6538 2900 50  0001 C CNN
 F 3 "" H 6500 3050 50  0000 C CNN
 	1    6500 3050
@@
 $EndComp
 $Comp
-L GND #PWR17
+L GND #PWR011
 U 1 1 5781095D
 P 6500 3250
-F 0 "#PWR17" H 6500 3000 50  0001 C CNN
+F 0 "#PWR011" H 6500 3000 50  0001 C CNN
 F 1 "GND" H 6500 3100 50  0000 C CNN
 F 2 "" H 6500 3250 50  0000 C CNN
@@
 $EndComp
 $Comp
-L +3.3V #PWR16
+L +3.3V #PWR012
 U 1 1 5781097A
 P 6500 2850
-F 0 "#PWR16" H 6500 2700 50  0001 C CNN
+F 0 "#PWR012" H 6500 2700 50  0001 C CNN
 F 1 "+3.3V" H 6500 2990 50  0000 C CNN
 F 2 "" H 6500 2850 50  0000 C CNN
@@
 F 0 "R1" H 1980 2750 50  0000 C CNN
 F 1 "DNP" V 1900 2750 50  0000 C CNN
-F 2 "" V 1830 2750 50  0000 C CNN
+F 2 "Resistors_SMD:R_0603" V 1830 2750 50  0001 C CNN
 F 3 "" H 1900 2750 50  0000 C CNN
 	1    1900 2750
@@
 F 0 "R2" H 2180 2750 50  0000 C CNN
 F 1 "DNP" V 2100 2750 50  0000 C CNN
-F 2 "" V 2030 2750 50  0000 C CNN
+F 2 "Resistors_SMD:R_0603" V 2030 2750 50  0001 C CNN
 F 3 "" H 2100 2750 50  0000 C CNN
 	1    2100 2750
@@
 $EndComp
 $Comp
-L +3.3V #PWR3
+L +3.3V #PWR013
 U 1 1 57810D5D
 P 2000 2500
-F 0 "#PWR3" H 2000 2350 50  0001 C CNN
+F 0 "#PWR013" H 2000 2350 50  0001 C CNN
 F 1 "+3.3V" H 2000 2640 50  0000 C CNN
 F 2 "" H 2000 2500 50  0000 C CNN
@@
 F 0 "R3" H 3930 2900 50  0000 C CNN
 F 1 "4.7k" V 3850 2900 50  0000 C CNN
-F 2 "" V 3780 2900 50  0000 C CNN
+F 2 "Resistors_SMD:R_0603" V 3780 2900 50  0001 C CNN
 F 3 "" H 3850 2900 50  0000 C CNN
 	1    3850 2900
@@
 $EndComp
 $Comp
-L +3.3V #PWR4
+L +3.3V #PWR014
 U 1 1 57811234
 P 3850 2700
-F 0 "#PWR4" H 3850 2550 50  0001 C CNN
+F 0 "#PWR014" H 3850 2550 50  0001 C CNN
 F 1 "+3.3V" H 3850 2840 50  0000 C CNN
 F 2 "" H 3850 2700 50  0000 C CNN
@@
 F 0 "U2" H 4900 3350 60  0000 C CNN
 F 1 "MCP9808" H 5250 2650 60  0000 C CNN
-F 2 "" H 5150 3050 60  0000 C CNN
+F 2 "Housings_DFN_QFN:DFN-8-1EP_3x2mm_Pitch0.5mm" H 5150 3050 60  0001 C CNN
 F 3 "" H 5150 3050 60  0000 C CNN
 	1    5150 3050
@@
 F 0 "U3" H 4900 5100 60  0000 C CNN
 F 1 "ABPMANN030PG2A3" H 5300 4600 60  0000 C CNN
-F 2 "" H 5150 4850 60  0000 C CNN
+F 2 "footprint:ABPMANN030PG2A3" H 5150 4850 60  0001 C CNN
 F 3 "" H 5150 4850 60  0000 C CNN
 	1    5150 4850
@@
 $EndComp
 $Comp
-L GND #PWR10
+L GND #PWR015
 U 1 1 57811DA0
 P 4600 5050
-F 0 "#PWR10" H 4600 4800 50  0001 C CNN
+F 0 "#PWR015" H 4600 4800 50  0001 C CNN
 F 1 "GND" H 4600 4900 50  0000 C CNN
 F 2 "" H 4600 5050 50  0000 C CNN
@@
 $EndComp
 $Comp
-L +3.3V #PWR9
+L +3.3V #PWR016
 U 1 1 57811DF1
 P 4600 4650
-F 0 "#PWR9" H 4600 4500 50  0001 C CNN
+F 0 "#PWR016" H 4600 4500 50  0001 C CNN
 F 1 "+3.3V" H 4600 4790 50  0000 C CNN
 F 2 "" H 4600 4650 50  0000 C CNN
@@
 F 0 "R4" H 4280 4550 50  0000 C CNN
 F 1 "4.7k" V 4200 4550 50  0000 C CNN
-F 2 "" V 4130 4550 50  0000 C CNN
+F 2 "Resistors_SMD:R_0603" V 4130 4550 50  0001 C CNN
 F 3 "" H 4200 4550 50  0000 C CNN
 	1    4200 4550
@@
 	4200 4750 4200 4700
 $Comp
-L +3.3V #PWR7
+L +3.3V #PWR017
 U 1 1 578124D1
 P 4200 4350
-F 0 "#PWR7" H 4200 4200 50  0001 C CNN
+F 0 "#PWR017" H 4200 4200 50  0001 C CNN
 F 1 "+3.3V" H 4200 4490 50  0000 C CNN
 F 2 "" H 4200 4350 50  0000 C CNN
@@
 F 0 "C4" H 6525 5000 50  0000 L CNN
 F 1 "0.1u" H 6525 4800 50  0000 L CNN
-F 2 "" H 6538 4750 50  0000 C CNN
+F 2 "Capacitors_SMD:C_0603" H 6538 4750 50  0001 C CNN
 F 3 "" H 6500 4900 50  0000 C CNN
 	1    6500 4900
@@
 $EndComp
 $Comp
-L GND #PWR19
+L GND #PWR018
 U 1 1 5781279D
 P 6500 5100
-F 0 "#PWR19" H 6500 4850 50  0001 C CNN
+F 0 "#PWR018" H 6500 4850 50  0001 C CNN
 F 1 "GND" H 6500 4950 50  0000 C CNN
 F 2 "" H 6500 5100 50  0000 C CNN
@@
 $EndComp
 $Comp
-L +3.3V #PWR18
+L +3.3V #PWR019
 U 1 1 578127A3
 P 6500 4700
-F 0 "#PWR18" H 6500 4550 50  0001 C CNN
+F 0 "#PWR019" H 6500 4550 50  0001 C CNN
 F 1 "+3.3V" H 6500 4840 50  0000 C CNN
 F 2 "" H 6500 4700 50  0000 C CNN
